Commit message: support both sim and real robot

File: description/robot.urdf.xacro (robot description, xacro)
@@ -1,11 +1,19 @@
 <?xml version="1.0"?>
 <robot xmlns:xacro="http://www.ros.org/wiki/xacro"  name="robot">
+    <!--
+    <xacro:arg name="use_ros2_control" default="true"/>
+    <xacro:arg name="sim_mode" default="false"/>
+    -->
+    <xacro:arg name="use_ros2_control" default="false"/>
+    <xacro:arg name="sim_mode" default="true"/>
     <xacro:include filename="robot_core.xacro" />
     <xacro:include filename="lidar.xacro" />
     <xacro:include filename="camera.xacro" />
-    <!-- control scheme-->
-    <!-- basic gazebo control using plan topics-->
-    <!-- <xacro:include filename="gazebo_control.xacro" /> -->
-    <!-- Ros2 control -->
-    <xacro:include filename="ros2_control.xacro" />
+    <!-- selecting what to run Gazebo or reak robot-->
+    <xacro:if value="$(arg use_ros2_control)">
+        <xacro:include filename="ros2_control.xacro" />
+    </xacro:if>
+    <xacro:unless value="$(arg use_ros2_control)">
+        <xacro:include filename="gazebo_control.xacro" />
+    </xacro:unless>
 </robot>

File: description/ros2_control.xacro (robot description, xacro)
@@ -1,13 +1,20 @@
 <?xml version="1.0"?>
 <robot xmlns:xacro="http://www.ros.org/wiki/xacro">
-<!-- This file add gazebo control plugins -->
-<ros2_control name="GazeboSystem" type="system">
+    <xacro:unless value="$(arg sim_mode)">
+        <ros2_control name="RealRobot" type="system">
     <hardware>
-        <plugin>gazebo_ros2_control/GazeboSystem</plugin>
+        <plugin>diffdrive_arduino/DiffDriveArduino</plugin>
+        <param name="left_wheel_name">left_wheel_joint</param>
+        <param name="right_wheel_name">right_wheel_joint</param>
+        <param name="loop_rate">10</param>
+        <param name="device">/dev/Arduino_UNO</param>
+        <param name="baud_rate">57600</param>
+        <param name="timeout">1000</param>
+        <param name="enc_counts_per_rev">80</param>
     </hardware>
     <joint name="left_wheel_joint">
         <command_interface name="velocity">
-            <param name="min">-10</param>
-            <param name="max">10</param>
+            <param name="min">-20</param>
+            <param name="max">20</param>
         </command_interface>
         <state_interface name="position" />
@@ -16,6 +23,6 @@
     <joint name="right_wheel_joint">
         <command_interface name="velocity">
-            <param name="min">-10</param>
-            <param name="max">10</param>
+            <param name="min">-20</param>
+            <param name="max">20</param>
         </command_interface>
         <state_interface name="velocity" />
@@ -23,8 +30,33 @@
     </joint>
 </ros2_control>
-<gazebo>
-    <plugin filename="libgazebo_ros2_control.so" name="gazebo_ros2_control">
-        <parameters>$(find poc_2W_Robot)/config/my_controllers.yaml</parameters>
-    </plugin>
-</gazebo>
+    </xacro:unless>
+    <xacro:if value="$(arg sim_mode)">
+        <ros2_control name="GazeboSystem" type="system">
+            <hardware>
+                <plugin>gazebo_ros2_control/GazeboSystem</plugin>
+            </hardware>
+            <joint name="left_wheel_joint">
+                <command_interface name="velocity">
+                    <param name="min">-10</param>
+                    <param name="max">10</param>
+                </command_interface>
+                <state_interface name="velocity"/>
+                <state_interface name="position"/>
+            </joint>
+            <joint name="right_wheel_joint">
+                <command_interface name="velocity">
+                    <param name="min">-10</param>
+                    <param name="max">10</param>
+                </command_interface>
+                <state_interface name="velocity"/>
+                <state_interface name="position"/>
+            </joint>
+        </ros2_control>
+    </xacro:if>
+    <gazebo>
+        <plugin name="gazebo_ros2_control" filename="libgazebo_ros2_control.so">
+            <parameters>$(find poc_2W_Robot)/config/my_controllers.yaml</parameters>
+            <parameters>$(find poc_2W_Robot)/config/gaz_ros2_ctl_use_sim.yaml</parameters>
+        </plugin>
+    </gazebo>
 </robot>

Commit message: robot side code

File: description/robot.urdf.xacro (robot description, xacro)
@@ -1,10 +1,10 @@
 <?xml version="1.0"?>
 <robot xmlns:xacro="http://www.ros.org/wiki/xacro"  name="robot">
-    <!--
     <xacro:arg name="use_ros2_control" default="true"/>
     <xacro:arg name="sim_mode" default="false"/>
-    -->
+<!--
     <xacro:arg name="use_ros2_control" default="false"/>
     <xacro:arg name="sim_mode" default="true"/>
+-->
     <xacro:include filename="robot_core.xacro" />
     <xacro:include filename="lidar.xacro" />

File: description/robot_core.xacro (robot description, xacro)
@@ -21,4 +21,12 @@
     <!-- BASE LINK -->
     <link name="base_link">
+    </link>
+    <!-- BASE_FOOTPRINT LINK -->
+    <joint name="base_footprint_joint" type="fixed">
+        <parent link="base_link"/>
+        <child link="base_footprint"/>
+        <origin xyz="0 0 0" rpy="0 0 0"/>
+    </joint>
+    <link name="base_footprint">
     </link>
     <!-- CHASSIS LINK -->

File: description/ros2_control.xacro (robot description, xacro)
@@ -10,11 +10,11 @@
         <param name="device">/dev/Arduino_UNO</param>
         <param name="baud_rate">57600</param>
-        <param name="timeout">1000</param>
+        <param name="timeout">3600</param>
         <param name="enc_counts_per_rev">80</param>
     </hardware>
     <joint name="left_wheel_joint">
         <command_interface name="velocity">
-            <param name="min">-20</param>
-            <param name="max">20</param>
+            <param name="min">-10</param>
+            <param name="max">10</param>
         </command_interface>
         <state_interface name="position" />
@@ -23,6 +23,6 @@
     <joint name="right_wheel_joint">
         <command_interface name="velocity">
-            <param name="min">-20</param>
-            <param name="max">20</param>
+            <param name="min">-10</param>
+            <param name="max">10</param>
         </command_interface>
         <state_interface name="velocity" />
