Commit message: fixed launch files

File: description/lidar.xacro (robot description, xacro)
@@ -26,5 +26,5 @@
         <sensor name="laser" type="ray">
             <pose> 0 0 0 0 0 0 </pose>
-            <visualize>false</visualize>
+            <visualize>true</visualize>
             <update_rate>10</update_rate>
             <ray>

File: description/robot.urdf.xacro (robot description, xacro)
@@ -5,5 +5,5 @@
     <xacro:arg name="sim_mode" default="false"/>
     -->
-    <xacro:arg name="use_ros2_control" default="false"/>
+    <xacro:arg name="use_ros2_control" default="true"/>
     <xacro:arg name="sim_mode" default="true"/>
     <xacro:include filename="robot_core.xacro" />
@@ -14,4 +14,5 @@
         <xacro:include filename="ros2_control.xacro" />
     </xacro:if>
+    <!--Basic Gazebo control without ros2_control-->
     <xacro:unless value="$(arg use_ros2_control)">
         <xacro:include filename="gazebo_control.xacro" />

File: description/robot_core.xacro (robot description, xacro)
@@ -21,4 +21,12 @@
     <!-- BASE LINK -->
     <link name="base_link">
+    </link>
+    <!-- BASE_FOOTPRINT LINK -->
+    <joint name="base_footprint_joint" type="fixed">
+        <parent link="base_link"/>
+        <child link="base_footprint"/>
+        <origin xyz="0 0 0" rpy="0 0 0"/>
+    </joint>
+    <link name="base_footprint">
     </link>
     <!-- CHASSIS LINK -->

Commit message: nav2 changes

File: description/lidar.xacro (robot description, xacro)
@@ -4,5 +4,5 @@
         <parent link="chassis"/>
         <child link="laser_frame"/>
-        <origin xyz="0.1 0 0.175" rpy="0 0 0"/>
+        <origin xyz="0.1 0 0.175" rpy="0 0 ${pi}"/>
     </joint>
     <link name="laser_frame">

File: description/robot.urdf.xacro (robot description, xacro)
@@ -9,10 +9,12 @@
     <xacro:include filename="robot_core.xacro" />
     <xacro:include filename="lidar.xacro" />
+   <!--
     <xacro:include filename="camera.xacro" />
+    -->
     <!-- selecting what to run Gazebo or reak robot-->
     <xacro:if value="$(arg use_ros2_control)">
         <xacro:include filename="ros2_control.xacro" />
     </xacro:if>
-    <!--Basic Gazebo control without ros2_control-->
+    <!--Basic Gazebo control without ros2_control -->
     <xacro:unless value="$(arg use_ros2_control)">
         <xacro:include filename="gazebo_control.xacro" />

File: description/robot_core.xacro (robot description, xacro)
@@ -3,5 +3,5 @@
     <xacro:include filename="inertial_macros.xacro"/>
 <!--Parameters-->
-    <xacro:property name="wheel_radius" value="0.05" />`
+    <xacro:property name="wheel_radius" value="0.09" />`
     <material name="white">
         <color rgba="1 1 1 1" />
@@ -21,12 +21,4 @@
     <!-- BASE LINK -->
     <link name="base_link">
-    </link>
-    <!-- BASE_FOOTPRINT LINK -->
-    <joint name="base_footprint_joint" type="fixed">
-        <parent link="base_link"/>
-        <child link="base_footprint"/>
-        <origin xyz="0 0 0" rpy="0 0 0"/>
-    </joint>
-    <link name="base_footprint">
     </link>
     <!-- BASE_FOOTPRINT LINK -->

File: description/ros2_control.xacro (robot description, xacro)
@@ -2,5 +2,5 @@
 <robot xmlns:xacro="http://www.ros.org/wiki/xacro">
     <xacro:unless value="$(arg sim_mode)">
-        <ros2_control name="RealRobot" type="system">
+    <ros2_control name="RealRobot" type="system">
     <hardware>
         <plugin>diffdrive_arduino/DiffDriveArduino</plugin>
@@ -15,6 +15,6 @@
     <joint name="left_wheel_joint">
         <command_interface name="velocity">
-            <param name="min">-10</param>
-            <param name="max">10</param>
+            <param name="min">-7</param>
+            <param name="max">7</param>
         </command_interface>
         <state_interface name="position" />
@@ -23,6 +23,6 @@
     <joint name="right_wheel_joint">
         <command_interface name="velocity">
-            <param name="min">-10</param>
-            <param name="max">10</param>
+            <param name="min">-7</param>
+            <param name="max">7</param>
         </command_interface>
         <state_interface name="velocity" />
@@ -38,6 +38,6 @@
             <joint name="left_wheel_joint">
                 <command_interface name="velocity">
-                    <param name="min">-10</param>
-                    <param name="max">10</param>
+                    <param name="min">0</param>
+                    <param name="max">7</param>
                 </command_interface>
                 <state_interface name="velocity"/>
@@ -46,6 +46,6 @@
             <joint name="right_wheel_joint">
                 <command_interface name="velocity">
-                    <param name="min">-10</param>
-                    <param name="max">10</param>
+                    <param name="min">0</param>
+                    <param name="max">7</param>
                 </command_interface>
                 <state_interface name="velocity"/>

Commit message: adding robot2 initial files and whacker wheel

File: description/lidar.xacro (robot description, xacro)
@@ -4,5 +4,6 @@
         <parent link="chassis"/>
         <child link="laser_frame"/>
-        <origin xyz="0.1 0 0.175" rpy="0 0 ${pi}"/>
+        <!--origin xyz="0.1 0 0.175" rpy="0 0 ${pi}"/-->
+        <origin xyz="0.38 0 0.175" rpy="0 0 ${pi}"/>
     </joint>
     <link name="laser_frame">

File: description/robot2.urdf.xacro (robot description, xacro)
@@ -7,10 +7,10 @@
     <xacro:arg name="sim_mode" default="true"/>
 -->
-    <xacro:include filename="robot_core.xacro" />
+    <xacro:include filename="robot2_core.xacro" />
     <xacro:include filename="lidar.xacro" />
     <xacro:include filename="camera.xacro" />
-    <!-- selecting what to run Gazebo or reak robot-->
+    <!-- selecting what to run Gazebo or real robot-->
     <xacro:if value="$(arg use_ros2_control)">
-        <xacro:include filename="ros2_control.xacro" />
+        <xacro:include filename="ros2_control2.xacro" />
     </xacro:if>
     <!--Basic Gazebo control without ros2_control -->

File: description/robot2_core.xacro (robot description, xacro)
@@ -109,14 +109,14 @@
         <material>Gazebo/Blue</material>
     </gazebo>
-    <!-- CASTER WHEEL LINK -->
-    <joint name="caster_wheel_joint" type="fixed">
+    <!-- WEED WHACKER WHEEL LINK -->
+    <joint name="whacker_wheel_joint" type="continuous">
         <parent link="chassis"/>
-        <child link="caster_wheel"/>
+        <child link="whacker_wheel"/>
         <origin xyz="0.3 0 0"/>
     </joint>
-    <link name="caster_wheel">
+    <link name="whacker_wheel">
         <visual>
             <geometry>
-                <sphere radius="0.05"/>
+                <sphere radius="0.08"/>
             </geometry>
             <material name="black"/>
@@ -124,12 +124,12 @@
         <collision>
             <geometry>
-                <sphere radius="0.05"/>
+                <sphere radius="0.08"/>
             </geometry>
         </collision>
-        <xacro:inertial_sphere mass="0.1" radius="0.05">
+        <xacro:inertial_sphere mass="0.1" radius="0.08">
             <origin xyz="0 0 0" rpy="0 0 0"/>
         </xacro:inertial_sphere>
     </link>
-    <gazebo reference="caster_wheel">
+    <gazebo reference="whacker_wheel">
         <material>Gazebo/Black</material>
         <mu1 value="0.001"/>

File: description/ros2_control2.xacro (robot description, xacro)
@@ -12,5 +12,12 @@
         <param name="timeout">3600</param>
         <param name="enc_counts_per_rev">9500</param>
+        <param name="whacker_wheel_name">whacker_wheel_joint</param>
     </hardware>
+    <joint name="whacker_wheel_joint">
+        <command_interface name="velocity">
+            <param name="min">-7</param>
+            <param name="max">7</param>
+        </command_interface>
+    </joint>
     <joint name="left_wheel_joint">
         <command_interface name="velocity">
@@ -36,4 +43,10 @@
                 <plugin>gazebo_ros2_control/GazeboSystem</plugin>
             </hardware>
+            <joint name="whacker_wheel_joint">
+                <command_interface name="velocity">
+                    <param name="min">0</param>
+                    <param name="max">7</param>
+                </command_interface>
+            </joint>
             <joint name="left_wheel_joint">
                 <command_interface name="velocity">
@@ -56,5 +69,5 @@
     <gazebo>
         <plugin name="gazebo_ros2_control" filename="libgazebo_ros2_control.so">
-            <parameters>$(find poc_2W_Robot)/config/my_controllers.yaml</parameters>
+            <parameters>$(find poc_2W_Robot)/config/my_controllers2.yaml</parameters>
             <parameters>$(find poc_2W_Robot)/config/gaz_ros2_ctl_use_sim.yaml</parameters>
         </plugin>
