Commit message: adding latest robot2 description xacro

File: description/robot2.urdf.xacro (robot description, xacro)
@@ -7,10 +7,10 @@
     <xacro:arg name="sim_mode" default="true"/>
 -->
-    <xacro:include filename="robot2_core.xacro" />
-    <xacro:include filename="lidar.xacro" />
-    <xacro:include filename="camera.xacro" />
+    <xacro:include filename="robot2_core_v1.xacro" />
+    <!--xacro:include filename="lidar.xacro" /-->
+    <!--xacro:include filename="camera_v1.xacro" /-->
     <!-- selecting what to run Gazebo or real robot-->
     <xacro:if value="$(arg use_ros2_control)">
-        <xacro:include filename="ros2_control2.xacro" />
+        <xacro:include filename="ros2_control2_v1.xacro" />
     </xacro:if>
     <!--Basic Gazebo control without ros2_control -->

File: description/ros2_control2_v1.xacro (robot description, xacro)
@@ -5,8 +5,8 @@
     <hardware>
         <plugin>diffdrive_arduino/DiffDriveArduino</plugin>
-        <param name="left_wheel_name">left_wheel_joint</param>
-        <param name="right_wheel_name">right_wheel_joint</param>
+        <param name="left_wheel_name">left_rear_wheel_joint</param>
+        <param name="right_wheel_name">right_rear_wheel_joint</param>
         <param name="loop_rate">10</param>
-	<param name="device">/dev/ttyUSB0</param>
+	    <param name="device">/dev/ttyUSB0</param>
         <param name="baud_rate">57600</param>
         <param name="timeout">3600</param>
@@ -20,5 +20,5 @@
         </command_interface>
     </joint>
-    <joint name="left_wheel_joint">
+    <joint name="left_rear_wheel_joint">
         <command_interface name="velocity">
             <param name="min">-7</param>
@@ -28,5 +28,5 @@
         <state_interface name="velocity" />
     </joint>
-    <joint name="right_wheel_joint">
+    <joint name="right_rear_wheel_joint">
         <command_interface name="velocity">
             <param name="min">-7</param>
@@ -69,5 +69,5 @@
     <gazebo>
         <plugin name="gazebo_ros2_control" filename="libgazebo_ros2_control.so">
-            <parameters>$(find poc_2W_Robot)/config/my_controllers2.yaml</parameters>
+            <parameters>$(find poc_2W_Robot)/config/my_controllers2_v1.yaml</parameters>
             <parameters>$(find poc_2W_Robot)/config/gaz_ros2_ctl_use_sim.yaml</parameters>
         </plugin>
